Commit message: minor

File: catkin_ws/src/multi_robot_scenario/xacro/camera/cctv5.xacro (robot description, xacro)
@@ -2,5 +2,5 @@
     <link name="world"/>
     <joint name="world_joint" type="fixed">
-        <origin xyz="0.0 0 0" rpy="0 0.78535 5.49745"/>
+        <origin xyz="0.0 0 0" rpy="0 0.78535 0.0"/>
         <!--r: roll(왼쪽으로 기움), p(pitch) y: yaw(좌우), 양수일 수록 밑을 내려봄, 45도 좌로-->
         <parent link="world"/>
