Commit message: [ADDED]DWA as local navigation

File: catkin_ws/src/multi_robot_scenario/xacro/camera/cctv2.xacro (robot description, xacro)
@@ -2,5 +2,5 @@
     <link name="world"/>
     <joint name="world_joint" type="fixed">
-        <origin xyz="0.0 0 0" rpy="0 0.78535 0.78535"/>
+        <origin xyz="0.0 0 0" rpy="0 0.38535 0.78535*4"/>
         <!--r: roll(왼쪽으로 기움), p(pitch) y: yaw(좌우), 양수일 수록 밑을 내려봄, 45도 좌로-->
         <parent link="world"/>

File: catkin_ws/src/multi_robot_scenario/xacro/p3dx/pioneer3dx_plugins.xacro (robot description, xacro)
@@ -16,5 +16,5 @@
             <rosDebugLevel>Debug</rosDebugLevel>
             <robotNamespace></robotNamespace>
-            <publishWheelTF>false</publishWheelTF>
+            <publishWheelTF>true</publishWheelTF>
             <!--배속걸때 문제 생기는 부분. 이걸 true->false로 바꾸면 나아짐?--><!--https://blog.csdn.net/weixin_41070687/article/details/125736727-->
             <!--publishWheelJointState>true</publishWheelJointState-->

Commit message: fixed code

File: catkin_ws/src/multi_robot_scenario/xacro/camera/cctv2.xacro (robot description, xacro)
@@ -2,6 +2,7 @@
     <link name="world"/>
     <joint name="world_joint" type="fixed">
-        <origin xyz="0.0 0 0" rpy="0 0.38535 0.78535*4"/>
-        <!--r: roll(왼쪽으로 기움), p(pitch) y: yaw(좌우), 양수일 수록 밑을 내려봄, 45도 좌로-->
+        <origin xyz="0.0 0 0" rpy="0 0.592675 -1.5707"/>   <!--남쪽-->   <!--수식 안먹힘-->
+        <!--0.38535-->
+        <!--r: roll(왼쪽으로 기움), p(pitch) y: yaw(좌우), 양수일 수록 밑을 내려봄, 음수면 왼쪽-->
         <parent link="world"/>
         <child link="cctv2"/>

File: catkin_ws/src/multi_robot_scenario/xacro/camera/cctv3.xacro (robot description, xacro)
@@ -2,6 +2,5 @@
     <link name="world"/>
     <joint name="world_joint" type="fixed">
-        <origin xyz="0.0 0 0" rpy="0 0.78535 2.35605"/>
-        <!--r: roll(왼쪽으로 기움), p(pitch) y: yaw(좌우), 양수일 수록 밑을 내려봄, 45도 좌로-->
+        <origin xyz="0.0 0 0" rpy="0 0.592675 -1.5707"/>
         <parent link="world"/>
         <child link="cctv3"/>

File: catkin_ws/src/multi_robot_scenario/xacro/camera/cctv4.xacro (robot description, xacro)
@@ -2,6 +2,5 @@
     <link name="world"/>
     <joint name="world_joint" type="fixed">
-        <origin xyz="0.0 0 0" rpy="0 0.78535 3.92675"/>
-        <!--r: roll(왼쪽으로 기움), p(pitch) y: yaw(좌우), 양수일 수록 밑을 내려봄, 45도 좌로-->
+        <origin xyz="0.0 0 0" rpy="0 0.592675 -1.5707"/>
         <parent link="world"/>
         <child link="cctv4"/>

File: catkin_ws/src/multi_robot_scenario/xacro/camera/cctv5.xacro (robot description, xacro)
@@ -3,5 +3,4 @@
     <joint name="world_joint" type="fixed">
         <origin xyz="0.0 0 0" rpy="0 0.78535 0.0"/>
-        <!--r: roll(왼쪽으로 기움), p(pitch) y: yaw(좌우), 양수일 수록 밑을 내려봄, 45도 좌로-->
         <parent link="world"/>
         <child link="cctv5"/>
