Commit message: ICRA2023 final version code

File: catkin_ws/src/multi_robot_scenario/xacro/camera/cctv.xacro (robot description, xacro)
@@ -2,5 +2,5 @@
     <link name="world"/>
     <joint name="world_joint" type="fixed">
-        <origin xyz="0.0 0 0" rpy="-1.5707 1.5707 0"/>
+        <origin xyz="0.0 0 0" rpy="0 0.78535 0.2"/>
         <parent link="world"/>
         <child link="cctv1"/>

File: catkin_ws/src/multi_robot_scenario/xacro/camera/cctv2.xacro (robot description, xacro)
@@ -6,7 +6,7 @@
         <!--r: roll(왼쪽으로 기움), p(pitch) y: yaw(좌우), 양수일 수록 밑을 내려봄, 음수면 왼쪽-->
         <parent link="world"/>
-        <child link="cctv2"/>
+        <child link="cctv1"/>
     </joint>
-    <link name="cctv2">
+    <link name="cctv1">
         <visual>
             <origin xyz="0 0 0" rpy="0 0 0"/>
@@ -21,8 +21,8 @@
         </inertial>
     </link>
-    <gazebo reference="cctv2">
+    <gazebo reference="cctv1">
         <static>true</static>
         <turnGravityOff>true</turnGravityOff>
-        <sensor type="camera" name="cctv2">
+        <sensor type="camera" name="cctv1">
             <update_rate>30.0</update_rate>
             <camera name="head">
@@ -47,8 +47,8 @@
                 <alwaysOn>true</alwaysOn>
                 <updateRate>0.0</updateRate>
-                <cameraName>cctv2</cameraName>
-                <imageTopicName>/cctv2/image_raw</imageTopicName>
-                <cameraInfoTopicName>/cctv2/camera_info</cameraInfoTopicName>
-                <frameName>cctv2</frameName>
+                <cameraName>cctv1</cameraName>
+                <imageTopicName>/cctv1/image_raw</imageTopicName>
+                <cameraInfoTopicName>/cctv1/camera_info</cameraInfoTopicName>
+                <frameName>cctv1</frameName>
                 <hackBaseline>0.07</hackBaseline>
                 <distortionK1>0.0</distortionK1>

File: catkin_ws/src/multi_robot_scenario/xacro/camera/cctv3.xacro (robot description, xacro)
@@ -4,7 +4,7 @@
         <origin xyz="0.0 0 0" rpy="0 0.592675 -1.5707"/>
         <parent link="world"/>
-        <child link="cctv3"/>
+        <child link="cctv2"/>
     </joint>
-    <link name="cctv3">
+    <link name="cctv2">
         <visual>
             <origin xyz="0 0 0" rpy="0 0 0"/>
@@ -19,8 +19,8 @@
         </inertial>
     </link>
-    <gazebo reference="cctv3">
+    <gazebo reference="cctv2">
         <static>true</static>
         <turnGravityOff>true</turnGravityOff>
-        <sensor type="camera" name="cctv3">
+        <sensor type="camera" name="cctv2">
             <update_rate>30.0</update_rate>
             <camera name="head">
@@ -45,8 +45,8 @@
                 <alwaysOn>true</alwaysOn>
                 <updateRate>0.0</updateRate>
-                <cameraName>cctv3</cameraName>
-                <imageTopicName>/cctv3/image_raw</imageTopicName>
-                <cameraInfoTopicName>/cctv3/camera_info</cameraInfoTopicName>
-                <frameName>cctv3</frameName>
+                <cameraName>cctv2</cameraName>
+                <imageTopicName>/cctv2/image_raw</imageTopicName>
+                <cameraInfoTopicName>/cctv2/camera_info</cameraInfoTopicName>
+                <frameName>cctv2</frameName>
                 <hackBaseline>0.07</hackBaseline>
                 <distortionK1>0.0</distortionK1>

File: catkin_ws/src/multi_robot_scenario/xacro/camera/cctv4.xacro (robot description, xacro)
@@ -4,7 +4,7 @@
         <origin xyz="0.0 0 0" rpy="0 0.592675 -1.5707"/>
         <parent link="world"/>
-        <child link="cctv4"/>
+        <child link="cctv3"/>
     </joint>
-    <link name="cctv4">
+    <link name="cctv3">
         <visual>
             <origin xyz="0 0 0" rpy="0 0 0"/>
@@ -19,8 +19,8 @@
         </inertial>
     </link>
-    <gazebo reference="cctv4">
+    <gazebo reference="cctv3">
         <static>true</static>
         <turnGravityOff>true</turnGravityOff>
-        <sensor type="camera" name="cctv4">
+        <sensor type="camera" name="cctv3">
             <update_rate>30.0</update_rate>
             <camera name="head">
@@ -45,8 +45,8 @@
                 <alwaysOn>true</alwaysOn>
                 <updateRate>0.0</updateRate>
-                <cameraName>cctv4</cameraName>
-                <imageTopicName>/cctv4/image_raw</imageTopicName>
-                <cameraInfoTopicName>/cctv4/camera_info</cameraInfoTopicName>
-                <frameName>cctv4</frameName>
+                <cameraName>cctv3</cameraName>
+                <imageTopicName>/cctv3/image_raw</imageTopicName>
+                <cameraInfoTopicName>/cctv3/camera_info</cameraInfoTopicName>
+                <frameName>cctv3</frameName>
                 <hackBaseline>0.07</hackBaseline>
                 <distortionK1>0.0</distortionK1>
