Commit message: update

File: catkin_ws/src/multi_robot_scenario/xacro/camera/cctv3.xacro (robot description, xacro)
@@ -2,5 +2,5 @@
     <link name="world"/>
     <joint name="world_joint" type="fixed">
-        <origin xyz="0.0 0 0" rpy="0 0.592675 -1.5707"/>
+        <origin xyz="0.0 0 0" rpy="0 0.592675 0"/>
         <parent link="world"/>
         <child link="cctv2"/>
